File: PCB 2022 version/watch_game_2022_revB.sch (EAGLE design)
At the start: 44 parts, among them J1 1734510-1, Q1 32.768, U1 ATTINY1616-SNR, U2 MCP73832T-5ACI/OT

Commit message: initial conversion to platformio note - moon force works, mgc test app has a glitch
Parts:
- U3: device bt_regulator:LF50CDT -> bt_regulator:NCP5501DT33RKG
Changed lines of the file:
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@@
 <part name="BAT-" library="adafruit" deviceset="PINHD-1X1" device=""/>
 <part name="HORI" library="diy-modules" deviceset="DISPLAY-OLED-128X64_A" device=""/>
-<part name="U3" library="bt_regulator" deviceset="LF50CDT" device=""/>
+<part name="U3" library="bt_regulator" deviceset="NCP5501DT33RKG" device=""/>
 <part name="J1" library="USB 1734510-1" deviceset="1734510-1" device=""/>
 <part name="C4" library="rcl" library_urn="urn:adsk.eagle:library:334" deviceset="C-US" device="C0805" package3d_urn="urn:adsk.eagle:package:23617/2" value="1uf"/>
